Commit message: add randomized terrain

File: gym/envs/dart/assets/darwinmodel/ground1.urdf (robot description, URDF)
Before this commit: robot ground_skeleton, 7 links, 6 joints
Links:
- removed link ground_link2
- added link obstacle1, mass 1.0; collision box size=0.4 25 2.05; visual box size=0.4 25 2.05
- added link obstacle2, mass 1.0; collision box size=0.2 25 2.05; visual box size=0.2 25 2.05
- added link obstacle3, mass 1.0; collision box size=0.2 25 2.05; visual box size=0.2 25 2.05
- added link obstacle4, mass 1.0; collision box size=0.2 25 2.05; visual box size=0.2 25 2.05
- added link obstacle5, mass 1.0; collision box size=0.2 25 2.05; visual box size=0.2 25 2.05
Joints:
- removed joint ground_joint2
- added joint obstacle_joint1: type fixed, parent ground_link, child obstacle1, origin xyz=0 0 0 rpy=0 0 0
- added joint obstacle_joint2: type fixed, parent ground_link, child obstacle2, origin xyz=0 0 0 rpy=0 0 0
- added joint obstacle_joint3: type fixed, parent ground_link, child obstacle3, origin xyz=0 0 0 rpy=0 0 0
- added joint obstacle_joint4: type fixed, parent ground_link, child obstacle4, origin xyz=0 0 0 rpy=0 0 0
- added joint obstacle_joint5: type fixed, parent ground_link, child obstacle5, origin xyz=0 0 0 rpy=0 0 0

Commit message: bug fix and use narrower boards

File: gym/envs/dart/assets/darwinmodel/ground1.urdf (robot description, URDF)
Before this commit: robot ground_skeleton, 11 links, 10 joints
Links:
- added link obstacle6, mass 1.0; collision box size=0.1 25 2.05; visual box size=0.1 25 2.05
- added link obstacle7, mass 1.0; collision box size=0.1 25 2.05; visual box size=0.1 25 2.05
- link obstacle1: geometry collision box size=0.2 25 2.05; visual box size=0.2 25 2.05
- link obstacle2: geometry collision box size=0.1 25 2.05; visual box size=0.1 25 2.05
- link obstacle3: geometry collision box size=0.1 25 2.05; visual box size=0.1 25 2.05
- link obstacle4: geometry collision box size=0.1 25 2.05; visual box size=0.1 25 2.05
- link obstacle5: geometry collision box size=0.1 25 2.05; visual box size=0.1 25 2.05
Joints:
- added joint obstacle_joint6: type fixed, parent ground_link, child obstacle6, origin xyz=0 0 0 rpy=0 0 0
- added joint obstacle_joint7: type fixed, parent ground_link, child obstacle7, origin xyz=0 0 0 rpy=0 0 0
